File: schem/fpc.sch (EAGLE design)
At the start: 34 parts, among them IC1 74HC00N, IC10 74HC32N, IC2 74HC14N, IC3 74HC377N, IC4 74HC04N, IC5 74HC00N, IC6 74HC377N, IC7 74HC08N, IC8 74HC14N, IC9 74HC32N

Commit message: finished most schematics
Connections:
- removed net /CNT: IC7A.I0, IC7B.O
- removed net /RD: IC6A.4Q
- removed net /RD0: IC6A.4D, IC7A.O
- new net CNT: IC1C.O
- net /DEPN1: now also IC1C.I1; no longer IC7B.I1
- net /EXAM: no longer IC7A.I1
- net /EXAMN: now also IC1C.I0; no longer IC7B.I0
Changed lines of the file:
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@@
 <instance part="GND8" gate="1" x="180.34" y="-5.08"/>
 <instance part="IC4" gate="E" x="246.38" y="22.86"/>
-<instance part="IC7" gate="A" x="243.84" y="7.62"/>
-<instance part="IC7" gate="B" x="243.84" y="-5.08"/>
 <instance part="IC7" gate="C" x="243.84" y="-17.78"/>
 <instance part="IC7" gate="D" x="276.86" y="25.4"/>
@@
 <instance part="IC10" gate="C" x="63.5" y="-83.82"/>
 <instance part="IC10" gate="D" x="63.5" y="-96.52"/>
+<instance part="IC1" gate="C" x="243.84" y="-5.08"/>
 </instances>
 <busses>
@@
 <label x="71.12" y="-58.42" size="1.778" layer="95"/>
 </segment>
-<segment>
-<pinref part="IC7" gate="A" pin="I1"/>
-<wire x1="236.22" y1="5.08" x2="226.06" y2="5.08" width="0.1524" layer="91"/>
-<label x="226.06" y="5.08" size="1.778" layer="95"/>
-</segment>
 </net>
 <net name="/EXAMN" class="0">
@@
 </segment>
 <segment>
-<pinref part="IC7" gate="B" pin="I0"/>
 <wire x1="226.06" y1="-2.54" x2="236.22" y2="-2.54" width="0.1524" layer="91"/>
 <label x="226.06" y="-2.54" size="1.778" layer="95"/>
+<pinref part="IC1" gate="C" pin="I0"/>
 </segment>
 </net>
@@
 </segment>
 </net>
-<net name="/CNT" class="0">
-<segment>
-<pinref part="IC7" gate="B" pin="O"/>
+<net name="CNT" class="0">
+<segment>
 <wire x1="251.46" y1="-5.08" x2="264.16" y2="-5.08" width="0.1524" layer="91"/>
 <label x="251.46" y="-5.08" size="1.778" layer="95"/>
-</segment>
-<segment>
-<pinref part="IC7" gate="A" pin="I0"/>
-<wire x1="236.22" y1="10.16" x2="226.06" y2="10.16" width="0.1524" layer="91"/>
-<label x="226.06" y="10.16" size="1.778" layer="95"/>
+<pinref part="IC1" gate="C" pin="O"/>
 </segment>
 </net>
@@
 </segment>
 <segment>
-<pinref part="IC7" gate="B" pin="I1"/>
 <wire x1="236.22" y1="-7.62" x2="226.06" y2="-7.62" width="0.1524" layer="91"/>
 <label x="226.06" y="-7.62" size="1.778" layer="95"/>
-</segment>
-</net>
-<net name="/RD0" class="0">
-<segment>
-<pinref part="IC7" gate="A" pin="O"/>
-<wire x1="251.46" y1="7.62" x2="264.16" y2="7.62" width="0.1524" layer="91"/>
-<label x="251.46" y="7.62" size="1.778" layer="95"/>
-</segment>
-<segment>
-<pinref part="IC6" gate="A" pin="4D"/>
-<wire x1="180.34" y1="15.24" x2="167.64" y2="15.24" width="0.1524" layer="91"/>
-<label x="167.64" y="15.24" size="1.778" layer="95"/>
-</segment>
-</net>
-<net name="/RD" class="0">
-<segment>
-<pinref part="IC6" gate="A" pin="4Q"/>
-<wire x1="205.74" y1="15.24" x2="218.44" y2="15.24" width="0.1524" layer="91"/>
-<label x="205.74" y="15.24" size="1.778" layer="95"/>
-</segment>
-</net>
+<pinref part="IC1" gate="C" pin="I1"/>
+</segment>
+</net>

Commit message: more work on several fronts
Connections:
- removed net /DEPN4: IC10D.O
- removed net /WR: IC7C.O
- new net /FOE: IC4F.O
- new net /FWE: IC9D.O
- new net /FWR: IC4F.I, IC7C.O, IC9D.I0
- net /DEPN: now also IC10D.O
- net CLK: now also IC9D.I1
Changed lines of the file:
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@@
 <instance part="IC10" gate="D" x="63.5" y="-96.52"/>
 <instance part="IC1" gate="C" x="243.84" y="-5.08"/>
+<instance part="IC9" gate="D" x="243.84" y="-30.48"/>
+<instance part="IC4" gate="F" x="246.38" y="-43.18"/>
 </instances>
 <busses>
@@
 <label x="167.64" y="0" size="1.778" layer="95"/>
 </segment>
+<segment>
+<pinref part="IC9" gate="D" pin="I1"/>
+<wire x1="226.06" y1="-33.02" x2="236.22" y2="-33.02" width="0.1524" layer="91"/>
+<label x="226.06" y="-33.02" size="1.778" layer="95"/>
+</segment>
 </net>
 <net name="SEXAM3" class="0">
@@
 </segment>
 </net>
-<net name="/DEPN4" class="0">
-<segment>
-<pinref part="IC10" gate="D" pin="O"/>
-<wire x1="71.12" y1="-96.52" x2="83.82" y2="-96.52" width="0.1524" layer="91"/>
-<label x="71.12" y="-96.52" size="1.778" layer="95"/>
-</segment>
-</net>
 <net name="RESET2" class="0">
 <segment>
@@
 <label x="167.64" y="17.78" size="1.778" layer="95"/>
 </segment>
-</net>
-<net name="/WR" class="0">
+<segment>
+<pinref part="IC10" gate="D" pin="O"/>
+<wire x1="71.12" y1="-96.52" x2="83.82" y2="-96.52" width="0.1524" layer="91"/>
+<label x="71.12" y="-96.52" size="1.778" layer="95"/>
+</segment>
+</net>
+<net name="/FWR" class="0">
 <segment>
 <pinref part="IC7" gate="C" pin="O"/>
@@
 <label x="251.46" y="-17.78" size="1.778" layer="95"/>
 </segment>
+<segment>
+<pinref part="IC9" gate="D" pin="I0"/>
+<wire x1="236.22" y1="-27.94" x2="226.06" y2="-27.94" width="0.1524" layer="91"/>
+<label x="226.06" y="-27.94" size="1.778" layer="95"/>
+</segment>
+<segment>
+<pinref part="IC4" gate="F" pin="I"/>
+<wire x1="236.22" y1="-43.18" x2="226.06" y2="-43.18" width="0.1524" layer="91"/>
+<label x="226.06" y="-43.18" size="1.778" layer="95"/>
+</segment>
 </net>
 <net name="CNT" class="0">
@@
 </segment>
 </net>
+<net name="/FWE" class="0">
+<segment>
+<pinref part="IC9" gate="D" pin="O"/>
+<wire x1="251.46" y1="-30.48" x2="264.16" y2="-30.48" width="0.1524" layer="91"/>
+<label x="251.46" y="-30.48" size="1.778" layer="95"/>
+</segment>
+</net>
+<net name="/FOE" class="0">
+<segment>
+<pinref part="IC4" gate="F" pin="O"/>
+<wire x1="256.54" y1="-43.18" x2="264.16" y2="-43.18" width="0.1524" layer="91"/>
+<label x="259.08" y="-43.18" size="1.778" layer="95"/>
+</segment>
+</net>
