File: schem/fp1.sch (EAGLE design)
At the start: 24 parts, among them IC1 74HC377N, IC10 74HC377N, IC11 74HC08N, IC12 ULN2003AN, IC13 ULN2003AN, IC14 ULN2003AN, IC15 74HC14N, IC2 74HC244N, IC3 74HC377N, IC4 74HC244N, IC5 74HC244N, IC6 74HC244N, IC7 74HC32N, IC8 74HC244N, IC9 74HC244N

Commit message: more work on front panel boards
Parts:
- added SV1, SV10, SV3, SV4, SV6, SV9: (no value), con-lstb:MA08-1
- added SV11: (no value), con-lstb:MA10-2
- added SV2, SV5, SV7, SV8: (no value), con-lstb:MA06-1
- C2, C3: value (none) -> 1u
- IC10: value 74HC377N -> 74HC14N; device 74xx-eu:74HC377N -> 74xx-eu:74HC14N
- IC11: value 74HC08N -> ULN2003AN; device 74xx-eu:74HC08N -> uln-udn:ULN2003AN
- IC14: value ULN2003AN -> 74HC08N; device uln-udn:ULN2003AN -> 74xx-eu:74HC08N
- IC15: value 74HC14N -> 74HC32N; device 74xx-eu:74HC14N -> 74xx-eu:74HC32N
- IC7: value 74HC32N -> 74HC244N; device 74xx-eu:74HC32N -> 74xx-eu:74HC244N
- IC9: value 74HC244N -> 74HC377N; device 74xx-eu:74HC244N -> 74xx-eu:74HC377N
Connections:
- new net /IRQ: SV7.6
- new net SYNC: SV8.2
- net /ACTV: now also IC15B.I1, SV6.1; no longer IC7B.I1
- net /BOE: now also IC7A.Y2, IC7B.Y2; no longer IC6B.Y2, IC9A.Y2
- net /BUSACK: now also IC7B.G, IC8B.G, SV7.2; no longer IC9A.G, IC9B.G
- net /BUSREQ: now also IC15C.O, SV7.3; no longer IC7C.O
- net /BWE: now also IC7A.Y1, IC7B.Y1; no longer IC6B.Y1, IC9A.Y1
- net /DEP: now also IC14B.I0, SV6.2; no longer IC11B.I0
- net /DEPN: now also IC14B.I1, IC9A.3D, SV6.3; no longer IC10A.3D, IC11B.I1
- net /DEPN1: now also IC9A.3Q, SV6.4; no longer IC10A.3Q
- net /FOE: now also IC10F.O, IC7B.A2; no longer IC15F.O, IC9A.A2
- net /FWE: now also IC15D.O, IC7B.A1; no longer IC7D.O, IC9A.A1
- net /FWR: now also IC10F.I, IC14B.O, IC15D.I0, IC6B.G; no longer IC11B.O, IC15F.I, IC7D.I0, IC8A.G
- net /RESET1: now also IC10B.O, SV6.7; no longer IC15B.O
- net /SSINGLE3: now also IC10E.O, IC14A.I1; no longer IC11A.I1, IC15E.O
- net /WE: now also IC7A.A1, SV7.4; no longer IC6B.A1
- net /WR: now also SV6.8
- net BUSACK: now also IC7A.G, IC8A.G, SV7.1; no longer IC6B.G, IC8B.G
- net BUSREQ0: now also IC15B.O, IC15C.I0; no longer IC7B.O, IC7C.I0
- net CLK: now also IC15D.I1, IC9A.CLK, SV2.3; no longer IC10A.CLK, IC7D.I1
- net DB0: now also IC12.I1, SV3.1; no longer IC13.I1
- net DB1: now also IC12.I2, SV3.2; no longer IC13.I2
- net DB2: now also IC12.I3, SV3.3; no longer IC13.I3
- net DB3: now also IC12.I4, SV3.4; no longer IC13.I4
- net DB4: now also IC12.I5, IC6B.Y1, SV3.5; no longer IC13.I5, IC8A.Y1
- net DB5: now also IC12.I6, IC6B.Y2, SV3.6; no longer IC13.I6, IC8A.Y2
- net DB6: now also IC12.I7, IC6B.Y3, SV3.7; no longer IC13.I7, IC8A.Y3
- net DB7: now also IC13.I2, IC6B.Y4, SV3.8; no longer IC14.I2, IC8A.Y4
- net DBLI0: now also IC12.O1, SV11.9; no longer IC13.O1
- net DBLI1: now also IC12.O2, SV11.10; no longer IC13.O2
- net DBLI2: now also IC12.O3, SV11.11; no longer IC13.O3
- net DBLI3: now also IC12.O4, SV11.12; no longer IC13.O4
- net DBLI4: now also IC12.O5, SV11.13; no longer IC13.O5
- net DBLI5: now also IC12.O6, SV11.14; no longer IC13.O6
- net DBLI6: now also IC12.O7, SV11.15; no longer IC13.O7
- net DBLI7: now also IC13.O2, SV11.16; no longer IC14.O2
- net GND: now also IC11.GND, IC9A.G, SV2.4, SV2.5, SV2.6, SV5.4, SV5.5, SV5.6; no longer IC10A.G, IC14.GND
- net IB0: now also IC11.I1, SV1.1; no longer IC12.I1
- net IB1: now also IC11.I2, SV1.2; no longer IC12.I2
- net IB2: now also IC11.I3, SV1.3; no longer IC12.I3
- net IB3: now also IC11.I4, SV1.4; no longer IC12.I4
- net IB4: now also IC11.I5, SV1.5; no longer IC12.I5
- net IB5: now also IC11.I6, SV1.6; no longer IC12.I6
- net IB6: now also IC11.I7, SV1.7; no longer IC12.I7
- net IB7: now also IC13.I1, SV1.8; no longer IC14.I1
- net IBD2: now also SV9.5
- net IBD3: now also SV9.6
- net IBF0: now also IC8B.A1; no longer IC9B.A1
- net IBF1: now also IC8B.A2; no longer IC9B.A2
- net IBF2: now also IC8B.A3; no longer IC9B.A3
- net IBF3: now also IC8B.A4; no longer IC9B.A4
- net IBLI0: now also IC11.O1, SV11.1; no longer IC12.O1
- net IBLI1: now also IC11.O2, SV11.2; no longer IC12.O2
- net IBLI2: now also IC11.O3, SV11.3; no longer IC12.O3
- net IBLI3: now also IC11.O4, SV11.4; no longer IC12.O4
- net IBLI4: now also IC11.O5, SV11.5; no longer IC12.O5
- net IBLI5: now also IC11.O6, SV11.6; no longer IC12.O6
- net IBLI6: now also IC11.O7, SV11.7; no longer IC12.O7
- net IBLI7: now also IC13.O1, SV11.8; no longer IC14.O1
- net IBR0: now also IC8A.A1, SV8.3; no longer IC8B.A1
- net IBR1: now also IC8A.A2, SV8.4; no longer IC8B.A2
- net IBR2: now also IC8A.A3, SV8.5; no longer IC8B.A3
- net IBR3: now also IC8A.A4, SV8.6; no longer IC8B.A4
- net IBS0: now also IC8A.Y1, SV9.1; no longer IC9B.Y1
- net IBS1: now also IC8A.Y2, SV9.2; no longer IC9B.Y2
- net IBS2: now also IC8A.Y3, SV9.3; no longer IC9B.Y3
- net IBS3: now also IC8A.Y4, SV9.4; no longer IC9B.Y4
- net OB0: now also SV4.1
- net OB1: now also SV4.2
- net OB2: now also SV4.3
- net OB3: now also SV4.4
- net OB4: now also SV4.5
- net OB5: now also SV4.6
- net OB6: now also SV4.7
- net OB7: now also SV4.8
- net OBD2: now also SV9.7
- net OBD3: now also SV9.8
- net RESET: now also IC15A.O, IC15B.I0, SV8.1; no longer IC7A.O, IC7B.I0
- net RESET0: now also IC10A.I; no longer IC15A.I
- net RESET1: now also IC10A.O, IC10B.I, IC15A.I0; no longer IC15A.O, IC15B.I, IC7A.I0
- net SINGLE: now also IC14A.O, IC15C.I1; no longer IC11A.O, IC7C.I1
- net SRESET: now also SV6.5
- net SRESET0: now also IC10C.I; no longer IC15C.I
- net SRESET1: now also IC10C.O, IC15A.I1; no longer IC15C.O, IC7A.I1
- net SSINGLE: now also SV6.6
- net SSINGLE0: now also IC10D.I; no longer IC15D.I
- net SSINGLE1: now also IC10D.O, IC9A.1D; no longer IC10A.1D, IC15D.O
- net SSINGLE2: now also IC14A.I0, IC9A.1Q, IC9A.2D; no longer IC10A.1Q, IC10A.2D, IC11A.I0
- net SSINGLE3: now also IC10E.I, IC9A.2Q; no longer IC10A.2Q, IC15E.I
- net SW0: now also SV10.1
- net SW1: now also SV10.2
- net SW2: now also SV10.3
- net SW3: now also SV10.4
- net SW4: now also IC6B.A1, SV10.5; no longer IC8A.A1
- net SW5: now also IC6B.A2, SV10.6; no longer IC8A.A2
- net SW6: now also IC6B.A3, SV10.7; no longer IC8A.A3
- net SW7: now also IC6B.A4, SV10.8; no longer IC8A.A4
- net VCC: now also SV11.17, SV11.18, SV11.19, SV11.20, SV2.1, SV2.2, SV5.1, SV5.2, SV5.3
- net WR: now also IC7A.A2, SV7.5; no longer IC6B.A2
Other:
- moved on the sheet: IC12, IC13, IC6B, IC8A, IC8B
